File: beamline.kicad_pcb (KiCad board)
At the start: 2 copper layers, 10 parts, among them U1 OPAMP_5-pin_Generic

Commit message: adding stuff
Parts:
- added C4: Capacitor_NP, Capacitor_SMD:C_0603_1608Metric, F.Cu at (103.2, 93.7)
- added C5: 1u, Capacitor_SMD:C_0603_1608Metric, F.Cu at (108.7, 85.6)
- added C6: 0.1u, Capacitor_SMD:C_0603_1608Metric, F.Cu at (108.7, 84.0)
- added C7: 10p, Capacitor_SMD:C_0603_1608Metric, F.Cu at (112.6, 85.7)
- added J1: Conn_02x10_Socket, PCM_SparkFun-Connector:2x10_P2.54mm_Socket_Vertical_SMD, B.Cu at (110.7, 72.9)
- added R5: 2k, Resistor_SMD:R_0402_1005Metric, F.Cu at (110.1, 87.1)
- C1: value 100nF -> 100n; footprint Capacitor_THT:C_Disc_D3.0mm_W2.0mm_P2.50mm -> Capacitor_SMD:C_0603_1608Metric
- C2: value 10nF -> 10n; footprint Capacitor_THT:C_Disc_D3.0mm_W2.0mm_P2.50mm -> Capacitor_SMD:C_0603_1608Metric
- C3: value Capacitor_NP -> 1u; footprint Capacitor_THT:C_Disc_D3.0mm_W2.0mm_P2.50mm -> Capacitor_SMD:C_0603_1608Metric
- R1: value Resistor -> 10
- R2: value Resistor -> 1k
- R4: value Resistor -> 2k
- moved R3 39.9 mm to (101.8, 93.8), turned to -90 degrees
- moved U1 38.8 mm to (106.9, 93.0), turned to 90 degrees
- moved D2 33.8 mm to (107.1, 88.6), turned to -90 degrees
- moved R4 33.7 mm to (109.5, 88.8), turned to 90 degrees
- moved R1 28.1 mm to (113.5, 92.6), turned to 90 degrees
- moved R2 28.0 mm to (114.1, 90.0), turned to 90 degrees
- moved D1 27.3 mm to (118.2, 91.5), turned to 180 degrees
- moved C3 26.5 mm to (111.9, 89.9), turned to 180 degrees
- moved C1 25.7 mm to (110.4, 92.5), turned to -90 degrees
- moved C2 24.5 mm to (112.0, 92.5), turned to -90 degrees
Connections:
- net /V_ref renamed Net-(D2-K)
- net Net-(D1-K) renamed /Bias Voltage/HV
- R1 pad 1: /V_Bias (~45V) -> unconnected-(R1-Pad1)
- R3 pad 1: OUT -> Net-(U1--)
- R3 pad 2: Net-(U1--) -> Net-(C4-Pad2)
- U1 pad 1: OUT -> Net-(C4-Pad2)
Routing:
- net GND: track 0.00 -> 24.3 mm
- net /Bias Voltage/HV: track 0.00 -> 15.0 mm
- net Net-(D2-K): track 0.00 -> 12.0 mm
- net Net-(D2-C): track 0.00 -> 9.85 mm
- net /SiPM signal: track 0.00 -> 7.05 mm
- net Net-(U1--): track 0.00 -> 6.90 mm
- net Net-(C4-Pad2): track 0.00 -> 4.34 mm
Other:
- board outline added: 34 x 38.2 mm
