File: _restore_backup_2026-06-26T19-07-32-494/beamline.kicad_sch (KiCad schematic)
At the start: 15 parts, among them U1 OPAMP_5-pin_Generic, U2 LM4040 2.5V

Commit message: adding stuff
Parts:
- removed U2: LM4040 2.5V, Package_TO_SOT_SMD:SOT-23, symbol Reference_Voltage:LM4040DBZ-2.5
- C1, C2, C3, C5, C6: footprint Capacitor_THT:C_Disc_D3.0mm_W2.0mm_P2.50mm -> Capacitor_SMD:C_0603_1608Metric
- C4: value 0.1u -> Capacitor_NP; footprint Capacitor_THT:C_Disc_D3.0mm_W2.0mm_P2.50mm -> Capacitor_SMD:C_0603_1608Metric
- D1: footprint Library:AFBRS4N44P014M -> AFBRS4N44P014M; symbol New_Library:AFBR-S4N44P014M -> New_Library:AFBR-S4N44P014MNUV-MT_Silicon_Photomultiplier; Height (none) -> 1.23; Manufacturer_Name (none) -> Avago Technologies; Manufacturer_Part_Number (none) -> AFBR-S4N44P014M; Mouser Part Number (none) -> 630-AFBR-S4N44P014M; Mouser Price/Stock (none) -> https://www.mouser.co.uk/ProductDetail/Broadcom-Avago/AFBR-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
Connections:
- net SiPM signal: now also D1.5 (A); no longer D1.2 (A)
- net at C1.2, C2.2, D1.1 (K)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: now also D1.2 (K), D1.3 (K), D1.4 (K)
- net +3.3V renamed +2.5V
Other:
- note removed: "Coaxial"
- moved on the sheet: C1, C2, C3, C4, C5, C6, R1, R2, R5
